Commit message: Realsense camera config file setup + rebuild

File: description/depth_camera.xacro (robot description, xacro)
@@ -2,6 +2,6 @@
 <robot xmlns:xacro="http://www.ros.org/wiki/xacro" >
     <joint name="camera_joint" type="fixed">
-        <parent link="chassis"/>
-        <child link="base_link"/>
+        <parent link="base_link"/>
+        <child link="camera_link"/>
         <origin xyz="0.37 0 0.08" rpy="0 0 0"/>
     </joint>
@@ -11,5 +11,5 @@
                 <box size="0.03 0.08 0.03"/>
             </geometry>
-            <material name="red"/>
+            <material name="orange"/>
         </visual>
     </link>

File: description/robot.urdf.xacro (robot description, xacro)
@@ -4,4 +4,5 @@
     <xacro:include filename = "robot_core.xacro"/>
     <xacro:include filename = "imu.xacro"/>
+    <xacro:include filename = "depth_camera.xacro"/>
     <xacro:include filename = "ros2_control.xacro"/>
 </robot>

Commit message: added depth camera to simulation

File: description/depth_camera.xacro (robot description, xacro)
@@ -4,5 +4,5 @@
         <parent link="base_link"/>
         <child link="camera_link"/>
-        <origin xyz="0.37 0 0.08" rpy="0 0 0"/>
+        <origin xyz="0.37 0 0.15" rpy="0 0 0"/>
     </joint>
     <link name="camera_link">
@@ -22,26 +22,44 @@
     <gazebo reference="camera_link">
         <material>Gazebo/Red</material>
-        <sensor name="camera" type="depth">
-            <pose> 0 0 0 0 0 0 </pose>
-            <visualize>true</visualize>
-            <update_rate>10</update_rate>
-            <camera>
-                <horizontal_fov>1.089</horizontal_fov>
+        <sensor name="camera" type="rgbd_camera">
+            <pose>0 0 0 0 0 0</pose>
+            <always_on>1</always_on>
+            <update_rate>30</update_rate>
+            <topic>camera</topic>
+            <visualize>1</visualize>
+            <enable_metrics>1</enable_metrics>
+            <gz_frame_id>camera_link_optical</gz_frame_id>
+            <camera name="camera">
+                <horizontal_fov>1.50098</horizontal_fov>
+                <distortion>
+                    <k1>0.0</k1>
+                    <k2>0.0</k2>
+                    <k3>0.0</k3>
+                    <p1>0.0</p1>
+                    <p2>0.0</p2>
+                    <center>0.5 0.5</center>
+                </distortion>
                 <image>
-                    <format>B8G8R8</format>
-                    <width>640</width>
+                    <width>848</width>
                     <height>480</height>
+                    <format>R8G8B8</format>
                 </image>
                 <clip>
-                    <near>0.05</near>
-                    <far>8.0</far>
+                    <near>0.1</near>
+                    <far>10.0</far>
                 </clip>
+                <depth_camera>
+                    <clip>
+                        <near>0.1</near>
+                        <far>10.0</far>
+                    </clip>
+                </depth_camera>
+                <noise>
+                    <type>gaussian</type>
+                    <mean>0</mean>
+                    <stddev>0.007</stddev>
+                </noise>
             </camera>
-            <plugin name="camera_controller" filename="libgazebo_ros_camera.so">
-                <frame_name>camera_link_optical</frame_name>
-                <min_depth>0.1</min_depth>
-                <max_depth>100.0</max_depth>
-            </plugin>
-        </sensor>
+      </sensor>
     </gazebo>
 </robot>

File: description/robot_core.xacro (robot description, xacro)
@@ -27,5 +27,5 @@
             <origin xyz="0.325 0 .075"/>
             <geometry>
-                <box size="0.65 0.43 0.15"/>
+                <box size="0.65 0.43 0.10"/>
             </geometry>
             <material name="white"/>

Commit message: xacro upates to handle some warnings

File: description/depth_camera.xacro (robot description, xacro)
@@ -20,4 +20,16 @@
     </joint>
     <link name="camera_link_optical"></link>
+    <joint name="d435i_joint" type="fixed">
+        <parent link="camera_link"/>
+        <child link="d435i_link"/>
+        <origin xyz="0 0 0" rpy="0 0 0"/>
+    </joint>
+    <link name="d435i_link"></link>
+    <joint name="d435i_camera_joint" type="fixed">
+        <parent link="camera_link"/>
+        <child link="d435i_camera_link"/>
+        <origin xyz="0 0 0" rpy="0 0 0"/>
+    </joint>
+    <link name="d435i_camera_link"></link>
     <gazebo reference="camera_link">
         <material>Gazebo/Red</material>

Commit message: depth to laser scan working. added mapping provisions in gazebo

File: description/depth_camera.xacro (robot description, xacro)
@@ -32,7 +32,14 @@
     </joint>
     <link name="d435i_camera_link"></link>
+    <joint name="camera_depth_joint" type="fixed">
+        <parent link="camera_link"/>
+        <child link="camera_depth_frame"/>
+        <origin xyz="0 0 0" rpy="0 0 0"/>
+    </joint>
+    <link name="camera_depth_frame"></link>
     <gazebo reference="camera_link">
         <material>Gazebo/Red</material>
-        <sensor name="camera" type="rgbd_camera">
+        <sensor name="camera_sensor" type="rgbd_camera">
+            <gz_frame_id>camera_link_optical</gz_frame_id>
             <pose>0 0 0 0 0 0</pose>
             <always_on>1</always_on>
@@ -41,5 +48,4 @@
             <visualize>1</visualize>
             <enable_metrics>1</enable_metrics>
-            <gz_frame_id>camera_link_optical</gz_frame_id>
             <camera name="camera">
                 <horizontal_fov>1.50098</horizontal_fov>
