Commit message: Added slam and exploration using nav2 to automatically create the map

File: description/robot_core.xacro (robot description, xacro)
@@ -16,4 +16,10 @@
     <!-- BASE LINK  -->
     <link name="base_link">
+    </link>
+    <joint name="base_footprint_joint" type="fixed">
+        <parent link="base_link"/>
+        <child link="base_footprint"/>
+    </joint>
+    <link name="base_footprint">
     </link>
     <!-- CHASSIS LINK -->
