Commit message: IMU running in sim mode

File: description/imu.xacro (robot description, xacro)
@@ -4,5 +4,5 @@
       <parent link="base_link"/>
       <child link="imu_link"/>
-      <origin xyz=".5 0 0" rpy="0 0 0"/>
+      <origin xyz=".1 0 0" rpy="0 0 0"/>
     </joint>
     <link name="imu_link">
@@ -20,3 +20,86 @@
       </collision>
     </link>
+    <xacro:if value="$(arg sim_mode)">
+      <gazebo reference="imu_link">
+        <sensor name="imu_sensor" type="imu">
+          <always_on>1</always_on>
+          <update_rate>50</update_rate>
+          <visualize>true</visualize>
+          <topic>imu</topic>
+          <imu>
+            <enable_orientation>0</enable_orientation>
+            <angular_velocity>
+              <x>
+                <!-- <noise type="gaussian">
+                  <mean>0</mean>
+                  <stddev>0.009</stddev>
+                  <bias_mean>0.00075</bias_mean>
+                  <bias_stddev>0.005</bias_stddev>
+                  <dynamic_bias_stddev>0.00002</dynamic_bias_stddev>
+                  <dynamic_bias_correlation_time>400.0</dynamic_bias_correlation_time>
+                  <precision>0.00025</precision>
+                </noise> -->
+              </x>
+              <y>
+                <!-- <noise type="gaussian">
+                  <mean>0</mean>
+                  <stddev>0.009</stddev>
+                  <bias_mean>0.00075</bias_mean>
+                  <bias_stddev>0.005</bias_stddev>
+                  <dynamic_bias_stddev>0.00002</dynamic_bias_stddev>
+                  <dynamic_bias_correlation_time>400.0</dynamic_bias_correlation_time>
+                  <precision>0.00025</precision>
+                </noise> -->
+              </y>
+              <z>
+                <!-- <noise type="gaussian">
+                  <mean>0</mean>
+                  <stddev>0.009</stddev>
+                  <bias_mean>0.00075</bias_mean>
+                  <bias_stddev>0.005</bias_stddev>
+                  <dynamic_bias_stddev>0.00002</dynamic_bias_stddev>
+                  <dynamic_bias_correlation_time>400.0</dynamic_bias_correlation_time>
+                  <precision>0.00025</precision>
+                </noise> -->
+              </z>
+            </angular_velocity>
+            <linear_acceleration>
+              <x>
+                <!-- <noise type="gaussian">
+                  <mean>0</mean>
+                  <stddev>0.021</stddev>
+                  <bias_mean>0.05</bias_mean>
+                  <bias_stddev>0.0075</bias_stddev>
+                  <dynamic_bias_stddev>0.000375</dynamic_bias_stddev>
+                  <dynamic_bias_correlation_time>175.0</dynamic_bias_correlation_time>
+                  <precision>0.005</precision>
+                </noise> -->
+              </x>
+              <y>
+                <!-- <noise type="gaussian">
+                  <mean>0</mean>
+                  <stddev>0.021</stddev>
+                  <bias_mean>0.05</bias_mean>
+                  <bias_stddev>0.0075</bias_stddev>
+                  <dynamic_bias_stddev>0.000375</dynamic_bias_stddev>
+                  <dynamic_bias_correlation_time>175.0</dynamic_bias_correlation_time>
+                  <precision>0.005</precision>
+                </noise> -->
+              </y>
+              <z>
+                <!-- <noise type="gaussian">
+                  <mean>0</mean>
+                  <stddev>0.021</stddev>
+                  <bias_mean>0.05</bias_mean>
+                  <bias_stddev>0.0075</bias_stddev>
+                  <dynamic_bias_stddev>0.000375</dynamic_bias_stddev>
+                  <dynamic_bias_correlation_time>175.0</dynamic_bias_correlation_time>
+                  <precision>0.005</precision>
+                </noise> -->
+              </z>
+            </linear_acceleration>
+          </imu>
+        </sensor>
+      </gazebo>
+    </xacro:if>
 </robot>

File: description/ros2_control.xacro (robot description, xacro)
@@ -57,5 +57,4 @@
         </joint>
     </ros2_control>
-    </xacro:if>
     <gazebo>
         <plugin name="gz_ros2_control::GazeboSimROS2ControlPlugin" filename="libgz_ros2_control-system.so">
@@ -64,3 +63,4 @@
         </plugin>
     </gazebo>
+    </xacro:if>
 </robot>

Commit message: updated IMU.xacro to precise location in the robot

File: description/imu.xacro (robot description, xacro)
@@ -4,5 +4,5 @@
       <parent link="base_link"/>
       <child link="imu_link"/>
-      <origin xyz=".1 0 0" rpy="0 0 0"/>
+      <origin xyz=".051 -.042 -0.024" rpy="0 ${pi/2} 0"/>
     </joint>
     <link name="imu_link">
